File: RCJ_Open_LinePCB.kicad_sch (KiCad schematic)
At the start: 205 parts, among them J1 Conn_01x12, U1 MCP3008, U2 MCP3008, U3 MCP3008, U4 MCP3008, U5 MCP3008, U6 MCP3008

Commit message: Completed Routing (No MCP)
Connections:
- net 3.3V: now also R37.1
Changed lines of the file:
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@@
+    )
+  )
+  (global_label "3.3V" (shape input) (at 276.225 60.96 90) (fields_autoplaced)
+    (effects (font (size 1.27 1.27)) (justify left))
+    (property "Intersheetrefs" "${INTERSHEET_REFS}" (at 276.3044 54.4345 90)
+      (effects (font (size 1.27 1.27)) (justify right) hide)
     )
   )

Commit message: Finished Routing
Routed all channel pins, all ADC pins, and header pins
Parts:
- U1, U2, U3, U4, U5, U6: footprint MCU-MCP3008-I_P_DIP16-7:MCP3008ISL -> MCP3008:SOIC16-N_MC_MCH-L
Changed lines of the file:
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@@
       (effects (font (size 1.27 1.27)) (justify right))
     )
-    (property "Footprint" "MCU-MCP3008-I_P_DIP16-7:MCP3008ISL" (at 269.875 206.375 0)
+    (property "Footprint" "MCP3008:SOIC16-N_MC_MCH-L" (at 269.875 206.375 0)
       (effects (font (size 1.27 1.27)) hide)
     )
@@
       (effects (font (size 1.27 1.27)) (justify right))
     )
-    (property "Footprint" "MCU-MCP3008-I_P_DIP16-7:MCP3008ISL" (at 46.355 200.025 0)
+    (property "Footprint" "MCP3008:SOIC16-N_MC_MCH-L" (at 46.355 200.025 0)
       (effects (font (size 1.27 1.27)) hide)
     )
@@
       (effects (font (size 1.27 1.27)) (justify right))
     )
-    (property "Footprint" "MCU-MCP3008-I_P_DIP16-7:MCP3008ISL" (at 214.63 205.74 0)
+    (property "Footprint" "MCP3008:SOIC16-N_MC_MCH-L" (at 214.63 205.74 0)
       (effects (font (size 1.27 1.27)) hide)
     )
@@
       (effects (font (size 1.27 1.27)) (justify right))
     )
-    (property "Footprint" "MCU-MCP3008-I_P_DIP16-7:MCP3008ISL" (at 160.02 201.93 0)
+    (property "Footprint" "MCP3008:SOIC16-N_MC_MCH-L" (at 160.02 201.93 0)
       (effects (font (size 1.27 1.27)) hide)
     )
@@
       (effects (font (size 1.27 1.27)) (justify right))
     )
-    (property "Footprint" "MCU-MCP3008-I_P_DIP16-7:MCP3008ISL" (at 101.6 200.025 0)
+    (property "Footprint" "MCP3008:SOIC16-N_MC_MCH-L" (at 101.6 200.025 0)
       (effects (font (size 1.27 1.27)) hide)
     )
@@
       (effects (font (size 1.27 1.27)) (justify right))
     )
-    (property "Footprint" "MCU-MCP3008-I_P_DIP16-7:MCP3008ISL" (at 329.565 208.915 0)
+    (property "Footprint" "MCP3008:SOIC16-N_MC_MCH-L" (at 329.565 208.915 0)
       (effects (font (size 1.27 1.27)) hide)
     )
